File: Hardware/Purpletooth_Jamboree.brd (EAGLE design)
At the start: 101.7 x 52.1 mm, 105 parts, among them Q1 MOSFET-NCHANNELBSS138, Q2 MOSFET-NCHANNELBSS138, Q3 MMBT4403, U2 MIC5219 3.3V, U3 TPA6138A2

Commit message: Replaced BC127 PKG w/ BC127_EXTRA_PASTE PKG
-Replaced the existing BC127 PKG with the BC127_EXTRA_PASTE PKG that
solved the cold-joint issues on the BC127 Module for the BC127 BOB (adds
extra paste to module pads).
-No hardware changes, just a stencil change.
Parts:
- U1: device SparkFun-RF:BC127 -> SparkFun-RF:BC127_XTRA_PASTE
Changed lines of the file:
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@@
 <?xml version="1.0" encoding="utf-8"?>
 <!DOCTYPE eagle SYSTEM "eagle.dtd">
-<eagle version="6.5.0">
+<eagle version="6.4">
 <drawing>
 <settings>
@@
 <setting verticaltext="up"/>
 </settings>
-<grid distance="0.05" unitdist="inch" unit="inch" style="lines" multiple="1" display="yes" altdistance="0.01" altunitdist="inch" altunit="inch"/>
+<grid distance="0.05" unitdist="inch" unit="inch" style="lines" multiple="1" display="yes" altdistance="0.005" altunitdist="inch" altunit="inch"/>
 <layers>
 <layer number="1" name="Top" color="4" fill="1" visible="yes" active="yes"/>
@@
 <layer number="19" name="Unrouted" color="6" fill="1" visible="yes" active="yes"/>
 <layer number="20" name="Dimension" color="6" fill="1" visible="yes" active="yes"/>
-<layer number="21" name="tPlace" color="6" fill="1" visible="yes" active="yes"/>
-<layer number="22" name="bPlace" color="6" fill="1" visible="yes" active="yes"/>
+<layer number="21" name="tPlace" color="16" fill="1" visible="yes" active="yes"/>
+<layer number="22" name="bPlace" color="14" fill="1" visible="yes" active="yes"/>
 <layer number="23" name="tOrigins" color="15" fill="1" visible="yes" active="yes"/>
 <layer number="24" name="bOrigins" color="15" fill="1" visible="yes" active="yes"/>
@@
 </autorouter>
 <elements>
-<element name="U1" library="SparkFun-RF" package="BC127" value="" x="54.61" y="41.91"/>
+<element name="U1" library="SparkFun-RF" package="BC127_XTRA_PASTE" value="" x="54.61" y="41.91"/>
 <element name="Q1" library="SparkFun-DiscreteSemi" package="SOT23" value="MOSFET-NCHANNELBSS138" x="68.58" y="40.64" rot="R270">
 <attribute name="PROD_ID" value="TRANS-00830" x="36.83" y="-11.43" size="1.778" layer="27" rot="R270" display="off"/>
