File: Hardware/Purpletooth_Jamboree.sch (EAGLE design)
At the start: 96 parts, among them Q1 MOSFET-NCHANNELBSS138, Q2 MOSFET-NCHANNELBSS138, Q3 MMBT4403, U2 MIC5219 3.3V

Commit message: Roll to next round of protos. - fix FTDI header pinouts - new USB footprint - add resistor to defeat charger temp sense - remove inductor to ground on audio input - fix buttons (add inline resistor, pull to 3.3v instead of ground) - add reset/pair2 button
Parts:
- removed L3: 15nH, SparkFun-Passives:INDUCTOR0603
- added JP21, JP22: M02PTH, SparkFun-Connectors:M02PTH
- added R27, R33: 10K, SparkFun-Resistors:10KOHM1/10W1%(0603)0603
- added R28, R29, R30, R31, R32: 2.2k, SparkFun-Resistors:2.2KOHM1/10W1%(0603)
- added S8: (no value), SparkFun-Electromechanical:TAC_SWITCHSMD
- JP2: value USB-MICROB -> USB_AB""; device SparkFun-Connectors:USB-MICROB -> SparkFun-Connectors:USB_AB""
- U3: PROD_ID (none) -> IC-11779
- renumbered U$1 to U3
Connections:
- removed net IN_GND: JP14.SLEEVE, JP18.3, L3.2
- new net N$1: JP21.2, R27.2, U3.!MUTE
- new net N$10: JP4.2, R28.1, S2.2
- new net N$11: JP5.2, R29.1, S3.2
- new net N$14: JP7.2, R30.1, S4.2
- new net N$15: JP8.2, R31.1, S5.2
- new net N$22: JP9.2, R32.1, S6.2
- net !RESET: now also JP22.2, S8.2
- net 3.3V: now also JP3.1, JP4.1, JP5.1, JP7.1, JP8.1, JP9.1, R27.1, S1.4, S2.4, S3.4, S4.4, S5.4, S6.4
- net 5V_RX: now also JP19.RXI; no longer JP19.TXO
- net 5V_TX: now also JP19.TXO; no longer JP19.RXI
- net AIO_1: now also R33.1
- net GND: now also JP14.SLEEVE, JP18.3, JP21.1, JP22.1, S8.4; no longer JP3.1, JP4.1, JP5.1, JP7.1, JP8.1, JP9.1, L3.1, S1.4, S2.4, S3.4, S4.4, S5.4, S6.4
- net PIO_0: now also R28.2; no longer JP4.2, S2.2
- net PIO_1: now also R29.2; no longer JP5.2, S3.2
- net PIO_2: now also R30.2; no longer JP7.2, S4.2
- net PIO_4: now also R31.2; no longer JP8.2, S5.2
- net PIO_5: now also R32.2; no longer JP9.2, S6.2
- net VIN: now also R33.2
Other:
- note added: "LONG: Become a source and connect to nearest or most recent sink."
- note added: "LONG: If sink, send CALL If source, initiate CALL"
- note added: "R33 is provided to allow battery to charge without a temp sensor."
- note added: "SHORT: Music back"
- note added: "SHORT: Music forward"
- note added: "SHORT: Play/pause Answer/end call"
- note added: "SHORT: Reset and become discoverable."
- note added: "SHORT: Volume down"
- note added: "SHORT: Volume up"
- note removed: "DOUBLE: Become a source and connect to nearest or most recent sink."
- note removed: "DOUBLE: If sink, send CALL If source, initiate CALL"
- note removed: "SINGLE: Music back"
- note removed: "SINGLE: Music forward"
- note removed: "SINGLE: Play/pause Answer/end call"
- note removed: "SINGLE: Reset and become discoverable."
- note removed: "SINGLE: Volume down"
- note removed: "SINGLE: Volume up"
- moved on the sheet: D1, D2, D3, JP10, JP11, JP15, JP16, JP3, JP4, JP5, JP7, JP8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

Commit message: Library update for connectors lib
Parts:
- JP2: value USB_AB"" -> (none); device SparkFun-Connectors:USB_AB"" -> SparkFun-Connectors:USB-ABCONN-11794
Changed lines of the file:
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@@
 <part name="GND12" library="SparkFun-Aesthetics" deviceset="GND" device=""/>
 <part name="FRAME2" library="SparkFun-Aesthetics" deviceset="FRAME-LETTER" device=""/>
-<part name="JP2" library="SparkFun-Connectors" deviceset="USB_AB" device="&quot;&quot;"/>
+<part name="JP2" library="SparkFun-Connectors" deviceset="USB-AB" device="CONN-11794"/>
 <part name="VIN2" library="SparkFun-Aesthetics" deviceset="5V" device="" value="V_USB"/>
 <part name="GND13" library="SparkFun-Aesthetics" deviceset="GND" device=""/>

Commit message: Transition to v10 for production - change labels on board and schematic - move top edge of board .05" up, to prevent module overhang from   interfering with panelization
Other:
- note added: "10"
- note removed: "01"
Changed lines of the file:
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@@
 <plain>
 <text x="172.72" y="7.62" size="3.81" layer="94">M. Hord</text>
-<text x="239.014" y="6.35" size="3.81" layer="94">01</text>
+<text x="239.014" y="6.35" size="3.81" layer="94">10</text>
 </plain>
 <instances>

Commit message: Added micro fiducial to board
Parts:
- removed FRAME2, FRAME3: FRAME-LETTER, SparkFun-Aesthetics:FRAME-LETTER
- added FID1, FID2: FIDUCIALUFIDUCIAL, SparkFun-Aesthetics:FIDUCIALUFIDUCIAL
Changed lines of the file:
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@@
 <?xml version="1.0" encoding="utf-8"?>
 <!DOCTYPE eagle SYSTEM "eagle.dtd">
-<eagle version="6.4">
+<eagle version="6.5.0">
 <drawing>
 <settings>
@@
 <part name="GND11" library="SparkFun-Aesthetics" deviceset="GND" device=""/>
 <part name="GND12" library="SparkFun-Aesthetics" deviceset="GND" device=""/>
-<part name="FRAME2" library="SparkFun-Aesthetics" deviceset="FRAME-LETTER" device=""/>
 <part name="JP2" library="SparkFun-Connectors" deviceset="USB-AB" device="CONN-11794"/>
 <part name="VIN2" library="SparkFun-Aesthetics" deviceset="5V" device="" value="V_USB"/>
 <part name="GND13" library="SparkFun-Aesthetics" deviceset="GND" device=""/>
 <part name="JP3" library="SparkFun-Connectors" deviceset="M02" device="PTH"/>
-<part name="FRAME3" library="SparkFun-Aesthetics" deviceset="FRAME-LETTER" device=""/>
 <part name="JP4" library="SparkFun-Connectors" deviceset="M02" device="PTH"/>
 <part name="JP5" library="SparkFun-Connectors" deviceset="M02" device="PTH"/>
@@
 <part name="SUPPLY21" library="SparkFun-Aesthetics" deviceset="5V" device="" value="VIN"/>
 <part name="GND21" library="SparkFun-Aesthetics" deviceset="GND" device=""/>
+<part name="FID1" library="SparkFun-Aesthetics" deviceset="FIDUCIAL" device="UFIDUCIAL"/>
+<part name="FID2" library="SparkFun-Aesthetics" deviceset="FIDUCIAL" device="UFIDUCIAL"/>
 </parts>
 <sheets>
@@
 <instance part="STANDOFF4" gate="G$1" x="246.38" y="33.02"/>
 <instance part="LOGO2" gate="G$1" x="88.9" y="0"/>
+<instance part="FID1" gate="G$1" x="152.4" y="38.1"/>
+<instance part="FID2" gate="G$1" x="157.48" y="38.1"/>
 </instances>
 <busses>
@@
 <instance part="GND11" gate="1" x="58.42" y="45.72"/>
 <instance part="GND12" gate="1" x="27.94" y="45.72"/>
-<instance part="FRAME2" gate="G$1" x="0" y="0"/>
-<instance part="FRAME2" gate="G$2" x="147.32" y="0"/>
 <instance part="S7" gate="G$1" x="83.82" y="27.94"/>
 <instance part="GND17" gate="1" x="93.98" y="15.24"/>
@@
 <instances>
 <instance part="JP3" gate="G$1" x="10.16" y="160.02"/>
-<instance part="FRAME3" gate="G$1" x="0" y="0"/>
-<instance part="FRAME3" gate="G$2" x="147.32" y="0"/>
 <instance part="U1" gate=".GPIO" x="180.34" y="127"/>
 <instance part="R2" gate="G$1" x="111.76" y="149.86" rot="R90"/>

Commit message: Replaced BC127 PKG w/ BC127_EXTRA_PASTE PKG
-Replaced the existing BC127 PKG with the BC127_EXTRA_PASTE PKG that
solved the cold-joint issues on the BC127 Module for the BC127 BOB (adds
extra paste to module pads).
-No hardware changes, just a stencil change.
Parts:
- U1: device SparkFun-RF:BC127 -> SparkFun-RF:BC127EXTRA_PASTE
Changed lines of the file:
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@@
 <?xml version="1.0" encoding="utf-8"?>
 <!DOCTYPE eagle SYSTEM "eagle.dtd">
-<eagle version="6.5.0">
+<eagle version="6.4">
 <drawing>
 <settings>
@@
 </classes>
 <parts>
-<part name="U1" library="SparkFun-RF" deviceset="BC127" device=""/>
+<part name="U1" library="SparkFun-RF" deviceset="BC127" device="EXTRA_PASTE"/>
 <part name="Q1" library="SparkFun-DiscreteSemi" deviceset="MOSFET-NCHANNEL" device="BSS138"/>
 <part name="U2" library="SparkFun-PowerIC" deviceset="V_REG_MIC5219" device="3.3V" value="MIC5219 3.3V"/>
